File: DFB1/kicad5/dfb1_r5/dfb1_r5.kicad_pcb (KiCad board)
At the start: 4 copper layers, 169 x 71.4 mm, 79 parts, among them IC1 IS42S16320D-7TL, IC2 IS42S16320D-7TL, IC3 SN74CB3T3245PW, IC4 SN74CB3T3245PW, IC5 SN74CB3T3245PW, IC6 SN74CB3T3245PW, J1 Conn_01x50, J2 Conn_02x04_Odd_Even, J3 Conn_01x30, J4 Conn_02x03_Odd_Even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

Commit message: Jumper labels updated to reflect production gerbers
Other:
- board text added: "DIS_FLASH"
- board text added: "OPTION1"
- board text added: "OPTION2"
- board text removed: "ALTRAM"
- board text removed: "FLASH"
- board text removed: "OPTION"
